File: Hardware/SoC/SparkFun_Dev_ESP32_C3.brd (EAGLE design)
At the start: 17.8 x 33 mm, 51 parts, among them J1 USB Female Type C Connector, J4 QWIIC_RIGHT_ANGLE, U1 ESP32-C3, U2 RT9080-33GJ5, Y1 40MHZ

Commit message: Adds MINI module, creates new design with MINI module netted
Parts:
- removed C6: 0.1uF, SparkFun-Capacitors:0402-TIGHT
- removed R8: 100k, SparkFun-Resistors:0402-TIGHT
- moved FD2 7.85 mm to (5.71, 25.5)
- moved D1 0.28 mm to (3.30, 31.9)
Connections:
- net 3.3V: no longer STAT.2
- net GND: no longer C6.2
- net IO9/BOOT: no longer C6.1
- net N$6: now also STAT.2; no longer R8.2, U2.3
- net V_USB: now also U2.3; no longer R8.1
