File: Hardware/SoC/SparkFun_Dev_ESP32_C3_PTH.brd (EAGLE design)
At the start: 17.8 x 33 mm, 49 parts, among them J1 USB Female Type C Connector, J4 QWIIC_RIGHT_ANGLE, U1 ESP32-C3_SOC, U2 RT9080-33GJ5, Y1 40MHZ

Commit message: Fixes symbol for ESP32 SOC, adds a few more headers, adds new SOC PTH design
Parts:
- removed J3: (no value), SparkFun-Connectors:1X12_CASTELLATED
- removed U$1: 1X10_CASTELLATED, ESP32-C3-MINI-1:1X10_CASTELLATED
- added J2: (no value), SparkFun-Connectors:1X10_NO_SILK
- added J6: (no value), SparkFun-Connectors:1X12_NO_SILK_KIT
- moved FD1 8.28 mm to (6.35, 25.4)
- moved E1 1.27 mm to (5.08, 1.27)
- moved FD2 0.65 mm to (6.35, 25.4)
Connections:
- net 3.3V: now also J6.4; no longer J3.4, J3.4B
- net EN: now also J6.3; no longer J3.3, J3.3B
- net GND: now also J2.7, J2.8, J6.2; no longer J3.2, J3.2B, U$1.7, U$1.7B, U$1.8, U$1.8B
- net IO0/A0: now also J6.8; no longer J3.8, J3.8B
- net IO1/A1: now also J6.7; no longer J3.7, J3.7B
- net IO10: now also J2.4; no longer U$1.4, U$1.4B
- net IO12: now also J2.3; no longer U$1.3, U$1.3B
- net IO13/SDA: now also J2.6; no longer U$1.6, U$1.6B
- net IO14/SCL: now also J2.5; no longer U$1.5, U$1.5B
- net IO15: now also J2.2; no longer U$1.2, U$1.2B
- net IO16: now also J2.1; no longer U$1.1, U$1.1B
- net IO2/POCI: now also J6.10; no longer J3.10, J3.10B
- net IO20/TXO: now also J2.10; no longer U$1.10, U$1.10B
- net IO21/RXI: now also J2.9; no longer U$1.9, U$1.9B
- net IO3/A3: now also J6.6; no longer J3.6, J3.6B
- net IO4/A4/MTMS: now also J6.5; no longer J3.5, J3.5B
- net IO5/A5/MTDI: now also J6.12; no longer J3.12, J3.12B
- net IO6/SCLK/MTCK: now also J6.9; no longer J3.9, J3.9B
- net IO7/PICO/MTDO: now also J6.11; no longer J3.11, J3.11B
- net V_USB: now also J6.1; no longer J3.1, J3.1B
