File: Hardware/SoC/SparkFun_Dev_ESP32_C3_PTH.sch (EAGLE design)
At the start: 48 parts, among them J1 USB Female Type C Connector, J4 QWIIC_RIGHT_ANGLE, U1 ESP32-C3_SOC, U2 RT9080-33GJ5, Y1 40MHZ

Commit message: Fixes symbol for ESP32 SOC, adds a few more headers, adds new SOC PTH design
Parts:
- removed J3: (no value), SparkFun-Connectors:CONN_12CASTELLATED
- removed U$1: 1X10_CASTELLATED, ESP32-C3-MINI-1:1X10_CASTELLATED
- added J2: (no value), SparkFun-Connectors:CONN_10NO_SILK_PTH_FEMALE
- added J6: (no value), SparkFun-Connectors:CONN_121X12_NO_SILK_KIT
Connections:
- net 3.3V: now also J6.4; no longer J3.4
- net EN: now also J6.3; no longer J3.3
- net GND: now also J2.7, J2.8, J6.2; no longer J3.2, U$1.7, U$1.8
- net IO0/A0: now also J6.8; no longer J3.8
- net IO1/A1: now also J6.7; no longer J3.7
- net IO10: now also J2.4; no longer U$1.4
- net IO12: now also J2.3; no longer U$1.3
- net IO13/SDA: now also J2.6; no longer U$1.6
- net IO14/SCL: now also J2.5; no longer U$1.5
- net IO15: now also J2.2; no longer U$1.2
- net IO16: now also J2.1; no longer U$1.1
- net IO2/POCI: now also J6.10; no longer J3.10
- net IO20/TXO: now also J2.10; no longer U$1.10
- net IO21/RXI: now also J2.9; no longer U$1.9
- net IO3/A3: now also J6.6; no longer J3.6
- net IO4/A4/MTMS: now also J6.5; no longer J3.5
- net IO5/A5/MTDI: now also J6.12; no longer J3.12
- net IO6/SCLK/MTCK: now also J6.9; no longer J3.9
- net IO7/PICO/MTDO: now also J6.11; no longer J3.11
- net V_USB: now also J6.1; no longer J3.1
Changed lines of the file:
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@@
 <part name="SUPPLY15" library="SparkFun-PowerSymbols" deviceset="3.3V" device=""/>
 <part name="GND16" library="SparkFun-PowerSymbols" deviceset="GND" device=""/>
-<part name="J3" library="SparkFun-Connectors" deviceset="CONN_12" device="CASTELLATED"/>
 <part name="SUPPLY16" library="SparkFun-PowerSymbols" deviceset="3.3V" device=""/>
 <part name="SUPPLY17" library="SparkFun-PowerSymbols" deviceset="V_USB" device=""/>
 <part name="GND18" library="SparkFun-PowerSymbols" deviceset="GND" device=""/>
 <part name="U1" library="ESP32-C3-MINI-1" deviceset="ESP32-C3_SOC" device=""/>
-<part name="U$1" library="ESP32-C3-MINI-1" deviceset="1X10_CASTELLATED" device=""/>
+<part name="J6" library="SparkFun-Connectors" deviceset="CONN_12" device="1X12_NO_SILK_KIT"/>
+<part name="J2" library="SparkFun-Connectors" deviceset="CONN_10" device="NO_SILK_PTH_FEMALE"/>
 </parts>
 <sheets>
@@
 <attribute name="VALUE" x="393.7" y="108.966" size="1.778" layer="96" font="vector" rot="MR0" align="top-center"/>
 </instance>
-<instance part="J3" gate="G$1" x="452.12" y="127" smashed="yes" rot="R180">
-<attribute name="VALUE" x="452.12" y="147.066" size="1.778" layer="96" font="vector" rot="R180"/>
-<attribute name="NAME" x="452.12" y="111.252" size="1.778" layer="95" font="vector" rot="R180"/>
-</instance>
 <instance part="SUPPLY16" gate="G$1" x="436.88" y="147.32" smashed="yes">
 <attribute name="VALUE" x="436.88" y="150.114" size="1.778" layer="96" font="vector" align="bottom-center"/>
@@
 <attribute name="VALUE" x="657.86" y="193.04" size="1.778" layer="96" font="vector"/>
 </instance>
-<instance part="U$1" gate="G$1" x="381" y="137.16" smashed="yes">
-<attribute name="VALUE" x="363.22" y="114.554" size="1.778" layer="96" font="vector"/>
+<instance part="J6" gate="G$1" x="452.12" y="127" smashed="yes" rot="R180">
+<attribute name="VALUE" x="452.12" y="147.066" size="1.778" layer="96" font="vector" rot="R180"/>
+<attribute name="NAME" x="452.12" y="111.252" size="1.778" layer="95" font="vector" rot="R180"/>
+</instance>
+<instance part="J2" gate="J1" x="381" y="137.16" smashed="yes">
+<attribute name="VALUE" x="381" y="114.554" size="1.778" layer="96" font="vector"/>
 <attribute name="NAME" x="381" y="145.288" size="1.778" layer="95" font="vector"/>
 </instance>
@@
 <wire x1="436.88" y1="134.62" x2="436.88" y2="147.32" width="0.1524" layer="91"/>
 <pinref part="SUPPLY16" gate="G$1" pin="3.3V"/>
-<pinref part="J3" gate="G$1" pin="4"/>
+<pinref part="J6" gate="G$1" pin="4"/>
 </segment>
 </net>
@@
 <junction x="393.7" y="134.62"/>
 <pinref part="GND16" gate="1" pin="GND"/>
-<pinref part="U$1" gate="G$1" pin="7"/>
-<pinref part="U$1" gate="G$1" pin="8"/>
+<pinref part="J2" gate="J1" pin="7"/>
+<pinref part="J2" gate="J1" pin="8"/>
 </segment>
 <segment>
@@
 <wire x1="439.42" y1="139.7" x2="439.42" y2="111.76" width="0.1524" layer="91"/>
 <pinref part="GND18" gate="1" pin="GND"/>
-<pinref part="J3" gate="G$1" pin="2"/>
+<pinref part="J6" gate="G$1" pin="2"/>
 </segment>
 </net>
@@
 <wire x1="429.26" y1="142.24" x2="429.26" y2="147.32" width="0.1524" layer="91"/>
 <pinref part="SUPPLY17" gate="G$1" pin="V_USB"/>
-<pinref part="J3" gate="G$1" pin="1"/>
+<pinref part="J6" gate="G$1" pin="1"/>
 </segment>
 </net>
@@
 <wire x1="441.96" y1="137.16" x2="434.34" y2="137.16" width="0.1524" layer="91"/>
 <label x="434.34" y="137.16" size="1.27" layer="95" font="vector" rot="R180" xref="yes"/>
-<pinref part="J3" gate="G$1" pin="3"/>
+<pinref part="J6" gate="G$1" pin="3"/>
 </segment>
 </net>
@@
 <wire x1="434.34" y1="129.54" x2="441.96" y2="129.54" width="0.1524" layer="91"/>
 <label x="434.34" y="129.54" size="1.27" layer="95" font="vector" rot="R180" xref="yes"/>
-<pinref part="J3" gate="G$1" pin="6"/>
+<pinref part="J6" gate="G$1" pin="6"/>
 </segment>
 </net>
@@
 <wire x1="391.16" y1="139.7" x2="396.24" y2="139.7" width="0.1524" layer="91"/>
 <label x="396.24" y="139.7" size="1.27" layer="95" font="vector" xref="yes"/>
-<pinref part="U$1" gate="G$1" pin="9"/>
+<pinref part="J2" gate="J1" pin="9"/>
 </segment>
 </net>
@@
 <wire x1="391.16" y1="142.24" x2="396.24" y2="142.24" width="0.1524" layer="91"/>
 <label x="396.24" y="142.24" size="1.27" layer="95" font="vector" xref="yes"/>
-<pinref part="U$1" gate="G$1" pin="10"/>
+<pinref part="J2" gate="J1" pin="10"/>
 </segment>
 </net>
@@
 <wire x1="434.34" y1="121.92" x2="441.96" y2="121.92" width="0.1524" layer="91"/>
 <label x="434.34" y="121.92" size="1.27" layer="95" font="vector" rot="R180" xref="yes"/>
-<pinref part="J3" gate="G$1" pin="9"/>
+<pinref part="J6" gate="G$1" pin="9"/>
 </segment>
 </net>
@@
 <wire x1="434.34" y1="119.38" x2="441.96" y2="119.38" width="0.1524" layer="91"/>
 <label x="434.34" y="119.38" size="1.27" layer="95" font="vector" rot="R180" xref="yes"/>
-<pinref part="J3" gate="G$1" pin="10"/>
+<pinref part="J6" gate="G$1" pin="10"/>
 </segment>
 </net>
@@
 <wire x1="434.34" y1="116.84" x2="441.96" y2="116.84" width="0.1524" layer="91"/>
 <label x="434.34" y="116.84" size="1.27" layer="95" font="vector" rot="R180" xref="yes"/>
-<pinref part="J3" gate="G$1" pin="11"/>
+<pinref part="J6" gate="G$1" pin="11"/>
 </segment>
 </net>
@@
 <wire x1="396.24" y1="132.08" x2="391.16" y2="132.08" width="0.1524" layer="91"/>
 <label x="396.24" y="132.08" size="1.27" layer="95" font="vector" xref="yes"/>
-<pinref part="U$1" gate="G$1" pin="6"/>
+<pinref part="J2" gate="J1" pin="6"/>
 </segment>
 </net>
@@
 <wire x1="396.24" y1="129.54" x2="391.16" y2="129.54" width="0.1524" layer="91"/>
 <label x="396.24" y="129.54" size="1.27" layer="95" font="vector" xref="yes"/>
-<pinref part="U$1" gate="G$1" pin="5"/>
+<pinref part="J2" gate="J1" pin="5"/>
 </segment>
 </net>
@@
 <wire x1="396.24" y1="121.92" x2="391.16" y2="121.92" width="0.1524" layer="91"/>
 <label x="396.24" y="121.92" size="1.27" layer="95" font="vector" xref="yes"/>
-<pinref part="U$1" gate="G$1" pin="2"/>
+<pinref part="J2" gate="J1" pin="2"/>
 </segment>
 </net>
@@
 <wire x1="434.34" y1="132.08" x2="441.96" y2="132.08" width="0.1524" layer="91"/>
 <label x="434.34" y="132.08" size="1.27" layer="95" font="vector" rot="R180" xref="yes"/>
-<pinref part="J3" gate="G$1" pin="5"/>
+<pinref part="J6" gate="G$1" pin="5"/>
 </segment>
 </net>
@@
 <wire x1="434.34" y1="127" x2="441.96" y2="127" width="0.1524" layer="91"/>
 <label x="434.34" y="127" size="1.27" layer="95" font="vector" rot="R180" xref="yes"/>
-<pinref part="J3" gate="G$1" pin="7"/>
+<pinref part="J6" gate="G$1" pin="7"/>
 </segment>
 </net>
@@
 <wire x1="434.34" y1="124.46" x2="441.96" y2="124.46" width="0.1524" layer="91"/>
 <label x="434.34" y="124.46" size="1.27" layer="95" font="vector" rot="R180" xref="yes"/>
-<pinref part="J3" gate="G$1" pin="8"/>
+<pinref part="J6" gate="G$1" pin="8"/>
 </segment>
 </net>
@@
 <wire x1="391.16" y1="127" x2="396.24" y2="127" width="0.1524" layer="91"/>
 <label x="396.24" y="127" size="1.27" layer="95" font="vector" xref="yes"/>
-<pinref part="U$1" gate="G$1" pin="4"/>
+<pinref part="J2" gate="J1" pin="4"/>
 </segment>
 </net>
@@
 <wire x1="396.24" y1="124.46" x2="391.16" y2="124.46" width="0.1524" layer="91"/>
 <label x="396.24" y="124.46" size="1.27" layer="95" font="vector" xref="yes"/>
-<pinref part="U$1" gate="G$1" pin="3"/>
+<pinref part="J2" gate="J1" pin="3"/>
 </segment>
 </net>
@@
 <wire x1="396.24" y1="119.38" x2="391.16" y2="119.38" width="0.1524" layer="91"/>
 <label x="396.24" y="119.38" size="1.27" layer="95" font="vector" xref="yes"/>
-<pinref part="U$1" gate="G$1" pin="1"/>
+<pinref part="J2" gate="J1" pin="1"/>
 </segment>
 </net>
@@
 <wire x1="434.34" y1="114.3" x2="441.96" y2="114.3" width="0.1524" layer="91"/>
 <label x="434.34" y="114.3" size="1.27" layer="95" font="vector" rot="R180" xref="yes"/>
-<pinref part="J3" gate="G$1" pin="12"/>
-</segment>
-</net>
+<pinref part="J6" gate="G$1" pin="12"/>
+</segment>
+</net>
