File: Hardware/Mini/SparkFun_Dev_ESP32_C3_MINI - PTH.brd (EAGLE design)
At the start: 17.8 x 33 mm, 44 parts, among them J1 USB Female Type C Connector, J5 Vertical Qwiic Connector, U2 RT9080-33GJ5

Commit message: Adds 9 pin connector to the MINI designs
Parts:
- removed J2, J3: (no value), SparkFun-Connectors:1X12_CASTELLATED
- added J4, J6: (no value), SparkFun-Connectors:1X09_NO_SILK
- moved LOGO2 10.8 mm to (5.08, 14.0), turned to 90 degrees
- moved FD1 7.85 mm to (5.71, 25.5)
- moved FD3 6.48 mm to (17.8, 6.35)
- moved FD4 6.48 mm to (17.8, 6.35)
- moved C9 1.27 mm to (17.8, 3.81)
- renumbered U$1 to U1
Connections:
- net 3.3V: now also J4.4; no longer J3.4, J3.4B
- net EN: now also J4.3; no longer J3.3, J3.3B
- net GND: now also J4.2, J6.3, J6.4; no longer J2.10, J2.10B, J2.9, J2.9B, J3.2, J3.2B
- net IO10: now also J6.9; no longer J2.4, J2.4B
- net IO20/TXO: now also J6.1; no longer J2.12, J2.12B
- net IO21/RXI: now also J6.2; no longer J2.11, J2.11B
- net IO5/SCL: now also J6.5; no longer J2.8, J2.8B
- net IO6/SDA: now also J6.6; no longer J2.7, J2.7B
- net IO7/STAT: now also J6.7; no longer J2.6, J2.6B
- net IO8: now also J6.8; no longer J2.5, J2.5B
- net IOA0/SCLK: now also J4.7; no longer J3.7, J3.7B
- net IOA1/POCI: now also J4.6; no longer J3.6, J3.6B
- net IOA2: now also J4.9; no longer J3.9, J3.9B
- net IOA3/PICO: now also J4.5; no longer J3.5, J3.5B
- net IOA4: now also J4.8; no longer J3.8, J3.8B
- net V_USB: now also J4.1; no longer J3.1, J3.1B
