File: Hardware/Mini/SparkFun_Dev_ESP32_C3_MINI - PTH.sch (EAGLE design)
At the start: 43 parts, among them J1 USB Female Type C Connector, J5 Vertical Qwiic Connector, U2 RT9080-33GJ5

Commit message: Adds 9 pin connector to the MINI designs
Parts:
- removed J2, J3: (no value), SparkFun-Connectors:CONN_12CASTELLATED
- added J4, J6: (no value), SparkFun-Connectors:CONN_09NO_SILK
- renumbered U$1 to U1
Connections:
- net 3.3V: now also J4.4; no longer J3.4
- net EN: now also J4.3; no longer J3.3
- net GND: now also J4.2, J6.3, J6.4; no longer J2.10, J2.9, J3.2
- net IO10: now also J6.9; no longer J2.4
- net IO20/TXO: now also J6.1; no longer J2.12
- net IO21/RXI: now also J6.2; no longer J2.11
- net IO5/SCL: now also J6.5; no longer J2.8
- net IO6/SDA: now also J6.6; no longer J2.7
- net IO7/STAT: now also J6.7; no longer J2.6
- net IO8: now also J6.8; no longer J2.5
- net IOA0/SCLK: now also J4.7; no longer J3.7
- net IOA1/POCI: now also J4.6; no longer J3.6
- net IOA2: now also J4.9; no longer J3.9
- net IOA3/PICO: now also J4.5; no longer J3.5
- net IOA4: now also J4.8; no longer J3.8
- net V_USB: now also J4.1; no longer J3.1
Other:
- note added: "Headers"
- note removed: "Castellated Headers"
