File: Hardware/Mini/SparkFun_Dev_ESP32_C3_MINI.brd (EAGLE design)
At the start: 17.8 x 33 mm, 44 parts, among them J1 USB Female Type C Connector, J5 Vertical Qwiic Connector, U2 RT9080-33GJ5

Commit message: Moves some parts away as lost in thought
Parts:
- moved C8 18.0 mm to (17.8, 2.54), turned to 0 degrees
- moved C9 15.5 mm to (17.8, 5.08), turned to 0 degrees
- moved R7 10.5 mm to (5.08, 12.7), turned to 180 degrees
- moved R3 2.84 mm to (12.7, 17.8), turned to 0 degrees
- moved R4 2.54 mm to (7.62, 17.8)
- moved C1 1.27 mm to (12.7, 21.6)
- moved C5 1.27 mm to (7.62, 20.3)
- moved R11 1.27 mm to (7.62, 21.6)
- moved R5 1.27 mm to (7.62, 22.9)
- moved R6 1.27 mm to (12.7, 22.9)
- moved R9 1.27 mm to (15.2, 17.8)

Commit message: Moves around some capacitors
Parts:
- moved R7 5.08 mm to (5.08, 17.8)
Changed lines of the file:
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@@
 <element name="LOGO2" library="SparkFun-Aesthetics" package="QWIIC_3MM" value="QWIIC_LOGO_3MM" x="12.7" y="6.35" smashed="yes"/>
 <element name="LOGO3" library="SparkFun-Aesthetics" package="OSHW-LOGO-S" value="OSHW-LOGOS" x="6.35" y="8.89" smashed="yes" rot="MR0"/>
-<element name="R7" library="SparkFun-Resistors" package="0402-TIGHT" value="100k" x="5.08" y="12.7" smashed="yes" rot="R180">
-<attribute name="NAME" x="5.08" y="12.138" size="0.6096" layer="25" font="vector" ratio="20" rot="R180" align="bottom-center"/>
-<attribute name="PROD_ID" value="RES-13495" x="5.08" y="12.7" size="1.778" layer="27" font="vector" ratio="15" rot="R180" display="off"/>
-<attribute name="VALUE" x="5.08" y="13.262" size="0.6096" layer="27" font="vector" ratio="20" rot="R180" align="top-center"/>
+<element name="R7" library="SparkFun-Resistors" package="0402-TIGHT" value="100k" x="5.08" y="17.78" smashed="yes" rot="R180">
+<attribute name="NAME" x="5.08" y="17.218" size="0.6096" layer="25" font="vector" ratio="20" rot="R180" align="bottom-center"/>
+<attribute name="PROD_ID" value="RES-13495" x="5.08" y="17.78" size="1.778" layer="27" font="vector" ratio="15" rot="R180" display="off"/>
+<attribute name="VALUE" x="5.08" y="18.342" size="0.6096" layer="27" font="vector" ratio="20" rot="R180" align="top-center"/>
 </element>
 <element name="R9" library="SparkFun-Resistors" package="0402-TIGHT" value="100k" x="15.24" y="17.78" smashed="yes">
@@
 <wire x1="17.78" y1="21.59" x2="19.35" y2="21.59" width="0" layer="19" extent="1-1"/>
 <wire x1="15.74" y1="17.78" x2="17.78" y2="21.59" width="0" layer="19" extent="1-1"/>
-<wire x1="4.58" y1="12.7" x2="15.74" y2="17.78" width="0" layer="19" extent="1-1"/>
-<wire x1="10.66" y1="15.735" x2="4.58" y2="12.7" width="0" layer="19" extent="1-1"/>
+<wire x1="4.58" y1="17.78" x2="15.74" y2="17.78" width="0" layer="19" extent="1-1"/>
+<wire x1="10.66" y1="15.735" x2="4.58" y2="17.78" width="0" layer="19" extent="1-1"/>
 <wire x1="10.16" y1="15.24" x2="10.66" y2="15.735" width="0" layer="19" extent="1-16"/>
 <wire x1="11.11" y1="20.2899" x2="10.66" y2="15.735" width="0" layer="19" extent="1-1"/>
@@
 <wire x1="7.12" y1="21.59" x2="11.11" y2="20.2899" width="0" layer="19" extent="1-1"/>
 <wire x1="3.1623" y1="31.75" x2="7.12" y2="21.59" width="0" layer="19" extent="1-16"/>
-<wire x1="16.06" y1="3.315" x2="4.58" y2="12.7" width="0" layer="19" extent="1-1"/>
+<wire x1="16.06" y1="3.315" x2="4.58" y2="17.78" width="0" layer="19" extent="1-1"/>
 </signal>
 <signal name="GND">
@@
 <contactref element="J2" pad="5"/>
 <contactref element="J2" pad="5B"/>
-<wire x1="6.96" y1="10.615" x2="5.58" y2="12.7" width="0" layer="19" extent="1-1"/>
+<wire x1="6.96" y1="10.615" x2="5.58" y2="17.78" width="0" layer="19" extent="1-1"/>
 <wire x1="2.54" y1="11.43" x2="6.96" y2="10.615" width="0" layer="19" extent="1-1"/>
 <wire x1="0.97" y1="11.43" x2="2.54" y2="11.43" width="0" layer="19" extent="1-1"/>

Commit message: Adds 9 pin connector to the MINI designs
Parts:
- removed J2, J3: (no value), SparkFun-Connectors:1X12_CASTELLATED
- added U$2, U$3: 1X09_CASTELLATED, ESP32-C3-MINI-1:1X09_CASTELLATED
- moved FD1 8.28 mm to (6.35, 25.4)
- moved C9 1.27 mm to (17.8, 3.81)
- moved FD2 0.65 mm to (6.35, 25.4)
Connections:
- net 3.3V: now also U$3.4, U$3.4B; no longer J3.4, J3.4B
- net EN: now also U$3.3, U$3.3B; no longer J3.3, J3.3B
- net GND: now also U$2.6, U$2.6B, U$2.7, U$2.7B, U$3.2, U$3.2B; no longer J2.10, J2.10B, J2.9, J2.9B, J3.2, J3.2B
- net IO10: now also U$2.1, U$2.1B; no longer J2.4, J2.4B
- net IO20/TXO: now also U$2.9, U$2.9B; no longer J2.12, J2.12B
- net IO21/RXI: now also U$2.8, U$2.8B; no longer J2.11, J2.11B
- net IO5/SCL: now also U$2.5, U$2.5B; no longer J2.8, J2.8B
- net IO6/SDA: now also U$2.4, U$2.4B; no longer J2.7, J2.7B
- net IO7/STAT: now also U$2.3, U$2.3B; no longer J2.6, J2.6B
- net IO8: now also U$2.2, U$2.2B; no longer J2.5, J2.5B
- net IOA0/SCLK: now also U$3.7, U$3.7B; no longer J3.7, J3.7B
- net IOA1/POCI: now also U$3.6, U$3.6B; no longer J3.6, J3.6B
- net IOA2: now also U$3.9, U$3.9B; no longer J3.9, J3.9B
- net IOA3/PICO: now also U$3.5, U$3.5B; no longer J3.5, J3.5B
- net IOA4: now also U$3.8, U$3.8B; no longer J3.8, J3.8B
- net V_USB: now also U$3.1, U$3.1B; no longer J3.1, J3.1B
