File: Hardware/SparkFun_Dev_ESP32_C3_MINI.sch (EAGLE design)
At the start: 43 parts, among them J1 USB Female Type C Connector, J5 Vertical Qwiic Connector, U2 RT9080-33GJ5

Commit message: Removes unnecessary documents, , moves boar daround
Connections:
- net IO10: now also U$2.2; no longer U$2.1
- net IO8: now also U$2.1; no longer U$2.2
Changed lines of the file:
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@@
 </segment>
 <segment>
-<wire x1="396.24" y1="124.46" x2="391.16" y2="124.46" width="0.1524" layer="91"/>
-<label x="396.24" y="124.46" size="1.27" layer="95" font="vector" xref="yes"/>
-<pinref part="U$2" gate="G$1" pin="2"/>
+<wire x1="396.24" y1="121.92" x2="391.16" y2="121.92" width="0.1524" layer="91"/>
+<label x="396.24" y="121.92" size="1.27" layer="95" font="vector" xref="yes"/>
+<pinref part="U$2" gate="G$1" pin="1"/>
 </segment>
 </net>
@@
 </segment>
 <segment>
-<wire x1="396.24" y1="121.92" x2="391.16" y2="121.92" width="0.1524" layer="91"/>
-<label x="396.24" y="121.92" size="1.27" layer="95" font="vector" xref="yes"/>
-<pinref part="U$2" gate="G$1" pin="1"/>
+<wire x1="396.24" y1="124.46" x2="391.16" y2="124.46" width="0.1524" layer="91"/>
+<label x="396.24" y="124.46" size="1.27" layer="95" font="vector" xref="yes"/>
+<pinref part="U$2" gate="G$1" pin="2"/>
 </segment>
 </net>

Commit message: Fixes net names that were blasted away
Connections:
- removed net IO7/STAT: STAT.2, TP1.1, U$1.IO7, U$2.3
- removed net IOA0/SCLK: U$1.IOA0, U$3.7
- removed net IOA1/POCI: U$1.IOA1, U$3.6
- removed net IOA3/PICO: TP4.1, U$1.IOA3, U$3.5
- removed net IOA4: U$1.IOA4, U$3.8
- new net IO7: U$1.IO7, U$2.3
- new net IOA0/SCLK/MTCK: TP3.1, U$1.IOA0, U$3.7
- new net IOA1/POCI/MTDO: STAT.2, TP1.1, U$1.IOA1, U$3.6
- new net IOA3/PICO/MTDI: TP6.1, U$1.IOA3, U$3.5
- new net IOA4/MTMS: TP4.1, U$1.IOA4, U$3.8
- net IO5/SCL: no longer TP6.1
- net IO6/SDA: no longer TP3.1
Changed lines of the file:
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@@
 </segment>
 </net>
-<net name="IO7/STAT" class="0">
-<segment>
-<wire x1="685.8" y1="215.9" x2="678.18" y2="215.9" width="0.1524" layer="91"/>
-<label x="685.8" y="215.9" size="1.27" layer="95" font="vector" xref="yes"/>
-<pinref part="U$1" gate="G$1" pin="IO7"/>
-</segment>
-<segment>
-<pinref part="TP1" gate="G$1" pin="1"/>
-<wire x1="403.86" y1="27.94" x2="408.94" y2="27.94" width="0.1524" layer="91" style="longdash"/>
-<label x="403.86" y="27.94" size="1.27" layer="95" font="vector" rot="R180" xref="yes"/>
-</segment>
-<segment>
-<wire x1="396.24" y1="127" x2="391.16" y2="127" width="0.1524" layer="91"/>
-<label x="396.24" y="127" size="1.27" layer="95" font="vector" rot="MR180" xref="yes"/>
-<pinref part="U$2" gate="G$1" pin="3"/>
-</segment>
-<segment>
-<pinref part="STAT" gate="G$1" pin="2"/>
-<wire x1="563.88" y1="66.04" x2="563.88" y2="68.58" width="0.1524" layer="91"/>
-<wire x1="563.88" y1="68.58" x2="566.42" y2="68.58" width="0.1524" layer="91"/>
-<label x="566.42" y="68.58" size="1.27" layer="95" font="vector" xref="yes"/>
-</segment>
-</net>
-<net name="IOA3/PICO" class="0">
-<segment>
-<pinref part="TP4" gate="G$1" pin="1"/>
-<wire x1="419.1" y1="17.78" x2="421.64" y2="17.78" width="0.1524" layer="91" style="longdash"/>
-<label x="421.64" y="17.78" size="1.27" layer="95" font="vector" xref="yes"/>
-</segment>
+<net name="IOA3/PICO/MTDI" class="0">
 <segment>
 <wire x1="685.8" y1="226.06" x2="678.18" y2="226.06" width="0.1524" layer="91"/>
@@
 <pinref part="U$3" gate="G$1" pin="5"/>
 </segment>
+<segment>
+<pinref part="TP6" gate="G$1" pin="1"/>
+<wire x1="419.1" y1="27.94" x2="421.64" y2="27.94" width="0.1524" layer="91" style="longdash"/>
+<label x="421.64" y="27.94" size="1.27" layer="95" font="vector" xref="yes"/>
+</segment>
 </net>
-<net name="IOA1/POCI" class="0">
+<net name="IOA1/POCI/MTDO" class="0">
 <segment>
 <wire x1="685.8" y1="231.14" x2="678.18" y2="231.14" width="0.1524" layer="91" style="longdash"/>
@@
 <pinref part="U$3" gate="G$1" pin="6"/>
 </segment>
+<segment>
+<pinref part="TP1" gate="G$1" pin="1"/>
+<wire x1="403.86" y1="27.94" x2="408.94" y2="27.94" width="0.1524" layer="91" style="longdash"/>
+<label x="403.86" y="27.94" size="1.27" layer="95" font="vector" rot="R180" xref="yes"/>
+</segment>
+<segment>
+<pinref part="STAT" gate="G$1" pin="2"/>
+<wire x1="563.88" y1="66.04" x2="563.88" y2="68.58" width="0.1524" layer="91"/>
+<wire x1="563.88" y1="68.58" x2="566.42" y2="68.58" width="0.1524" layer="91"/>
+<label x="566.42" y="68.58" size="1.27" layer="95" font="vector" xref="yes"/>
+</segment>
 </net>
-<net name="IOA0/SCLK" class="0">
+<net name="IOA0/SCLK/MTCK" class="0">
 <segment>
 <wire x1="685.8" y1="233.68" x2="678.18" y2="233.68" width="0.1524" layer="91" style="longdash"/>
@@
 <label x="436.88" y="127" size="1.27" layer="95" font="vector" rot="R180" xref="yes"/>
 <pinref part="U$3" gate="G$1" pin="7"/>
+</segment>
+<segment>
+<pinref part="TP3" gate="G$1" pin="1"/>
+<wire x1="408.94" y1="17.78" x2="403.86" y2="17.78" width="0.1524" layer="91" style="longdash"/>
+<label x="403.86" y="17.78" size="1.27" layer="95" font="vector" rot="R180" xref="yes"/>
 </segment>
 </net>
@@
 </segment>
 </net>
-<net name="IOA4" class="0">
+<net name="IOA4/MTMS" class="0">
 <segment>
 <wire x1="685.8" y1="223.52" x2="678.18" y2="223.52" width="0.1524" layer="91" style="longdash"/>
@@
 <pinref part="U$3" gate="G$1" pin="8"/>
 </segment>
+<segment>
+<pinref part="TP4" gate="G$1" pin="1"/>
+<wire x1="419.1" y1="17.78" x2="421.64" y2="17.78" width="0.1524" layer="91" style="longdash"/>
+<label x="421.64" y="17.78" size="1.27" layer="95" font="vector" xref="yes"/>
+</segment>
 </net>
 <net name="IO5/SCL" class="0">
@@
 <label x="426.72" y="76.2" size="1.27" layer="95" font="vector" xref="yes"/>
 <pinref part="J5" gate="J1" pin="4"/>
-</segment>
-<segment>
-<pinref part="TP6" gate="G$1" pin="1"/>
-<wire x1="419.1" y1="27.94" x2="421.64" y2="27.94" width="0.1524" layer="91" style="longdash"/>
-<label x="421.64" y="27.94" size="1.27" layer="95" font="vector" xref="yes"/>
 </segment>
 <segment>
@@
 </segment>
 <segment>
-<pinref part="TP3" gate="G$1" pin="1"/>
-<wire x1="408.94" y1="17.78" x2="403.86" y2="17.78" width="0.1524" layer="91" style="longdash"/>
-<label x="403.86" y="17.78" size="1.27" layer="95" font="vector" rot="R180" xref="yes"/>
-</segment>
-<segment>
 <wire x1="396.24" y1="129.54" x2="391.16" y2="129.54" width="0.1524" layer="91"/>
 <label x="396.24" y="129.54" size="1.27" layer="95" font="vector" rot="MR180" xref="yes"/>
@@
 </segment>
 </net>
+<net name="IO7" class="0">
+<segment>
+<wire x1="396.24" y1="127" x2="391.16" y2="127" width="0.1524" layer="91"/>
+<label x="396.24" y="127" size="1.27" layer="95" font="vector" rot="MR180" xref="yes"/>
+<pinref part="U$2" gate="G$1" pin="3"/>
+</segment>
+<segment>
+<wire x1="685.8" y1="215.9" x2="678.18" y2="215.9" width="0.1524" layer="91"/>
+<label x="685.8" y="215.9" size="1.27" layer="95" font="vector" xref="yes"/>
+<pinref part="U$1" gate="G$1" pin="IO7"/>
+</segment>
+</net>

Commit message: Adds I2S nets, we'll see
Connections:
- net IO10 renamed IO10/I2S_WS
- net IO5/SCL renamed IO5/SCL/BCK
- net IO6/SDA renamed IO6/SDA/I2S_SDO
- net IO7 renamed IO7/I2S_SDI
Changed lines of the file:
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@@
 </segment>
 </net>
-<net name="IO10" class="0">
+<net name="IO10/I2S_WS" class="0">
 <segment>
 <wire x1="685.8" y1="208.28" x2="678.18" y2="208.28" width="0.1524" layer="91" style="longdash"/>
@@
 </segment>
 </net>
-<net name="IO5/SCL" class="0">
+<net name="IO5/SCL/BCK" class="0">
 <segment>
 <wire x1="426.72" y1="76.2" x2="421.64" y2="76.2" width="0.1524" layer="91"/>
@@
 </segment>
 </net>
-<net name="IO6/SDA" class="0">
+<net name="IO6/SDA/I2S_SDO" class="0">
 <segment>
 <wire x1="421.64" y1="73.66" x2="426.72" y2="73.66" width="0.1524" layer="91"/>
@@
 </segment>
 </net>
-<net name="IO7" class="0">
+<net name="IO7/I2S_SDI" class="0">
 <segment>
 <wire x1="396.24" y1="127" x2="391.16" y2="127" width="0.1524" layer="91"/>

Commit message: Adds new C3 module so that the  device value is correct
* Fixes testpoints
Parts:
- renumbered U$1 to U1
Connections:
- removed net IOA1/POCI/MTDO: STAT.2, TP1.1, U$3.6, U1.IOA1
- removed net IOA3/PICO/MTDI: TP6.1, U$3.5, U1.IOA3
- new net IOA1/POCI/MTDI: STAT.2, TP6.1, U$3.6, U1.IOA1
- new net IOA3/PICO/MTDO: TP1.1, U$3.5, U1.IOA3
Other:
- moved on the sheet: TP1, TP2, TP3

Commit message: Moves stat LED
Connections:
- net IO10/I2S_WS: now also STAT.2
- net IOA1/POCI/MTDI: no longer STAT.2
Changed lines of the file:
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@@
-</segment>
-<segment>
-<pinref part="STAT" gate="G$1" pin="2"/>
-<wire x1="563.88" y1="66.04" x2="563.88" y2="68.58" width="0.1524" layer="91"/>
-<wire x1="563.88" y1="68.58" x2="566.42" y2="68.58" width="0.1524" layer="91"/>
-<label x="566.42" y="68.58" size="1.27" layer="95" font="vector" xref="yes"/>
 </segment>
 <segment>
@@
 <pinref part="U$2" gate="G$1" pin="2"/>
 </segment>
+<segment>
+<pinref part="STAT" gate="G$1" pin="2"/>
+<wire x1="563.88" y1="66.04" x2="563.88" y2="68.58" width="0.1524" layer="91"/>
+<wire x1="563.88" y1="68.58" x2="566.42" y2="68.58" width="0.1524" layer="91"/>
+<label x="566.42" y="68.58" size="1.27" layer="95" font="vector" xref="yes"/>
+</segment>
 </net>

Commit message: Renames some nets for clarity, adds vias, cleans up  ground pours, fixes air wires
Connections:
- net IO10/I2S_WS renamed IO10/I2S_FS
- net IO5/SCL/BCK renamed IO5/SCL/I2S_SCK
Changed lines of the file:
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@@
 </segment>
 </net>
-<net name="IO10/I2S_WS" class="0">
+<net name="IO10/I2S_FS" class="0">
 <segment>
 <wire x1="685.8" y1="208.28" x2="678.18" y2="208.28" width="0.1524" layer="91" style="longdash"/>
@@
 </segment>
 </net>
-<net name="IO5/SCL/BCK" class="0">
+<net name="IO5/SCL/I2S_SCK" class="0">
 <segment>
 <wire x1="426.72" y1="76.2" x2="421.64" y2="76.2" width="0.1524" layer="91"/>

Commit message: Adds more silk, removes some shield polygons on inner layers
* Moves fiducials around
* Swaps I2C lines at PTH header
Parts:
- removed C8: 0.1uF, SparkFun-Capacitors:0.1UF-0402T-16V-10%
- removed C9: 10uF, SparkFun-Capacitors:10UF-0402T-6.3V-20%
Connections:
- net 3.3V: no longer C8.1, C9.1
- net GND: no longer C8.2, C9.2
- net IO5/SCL/I2S_SCK: now also U$2.4; no longer U$2.5
- net IO6/SDA/I2S_SDO: now also U$2.5; no longer U$2.4
Other:
- note removed: "Digital Decoupling Pins 3"
Changed lines of the file:
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@@
 <setting verticaltext="up"/>
 </settings>
-<grid distance="0.1" unitdist="inch" unit="inch" style="lines" multiple="1" display="no" altdistance="0.01" altunitdist="inch" altunit="inch"/>
+<grid distance="0.5" unitdist="mm" unit="mm" style="lines" multiple="1" display="yes" altdistance="0.01" altunitdist="mm" altunit="mm"/>
 <layers>
 <layer number="1" name="Top" color="4" fill="1" visible="no" active="no"/>
@@
 <part name="GND21" library="SparkFun-PowerSymbols" deviceset="GND" device=""/>
 <part name="LOGO1" library="SparkFun-Aesthetics" deviceset="SFE_LOGO_NAME_FLAME" device="BLANK"/>
-<part name="C8" library="SparkFun-Capacitors" deviceset="0.1UF" device="-0402T-16V-10%" value="0.1uF"/>
-<part name="C9" library="SparkFun-Capacitors" deviceset="10UF" device="-0402T-6.3V-20%" value="10uF"/>
-<part name="GND9" library="SparkFun-PowerSymbols" deviceset="GND" device=""/>
-<part name="SUPPLY3" library="SparkFun-PowerSymbols" deviceset="3.3V" device=""/>
 <part name="JP14" library="SparkFun-Connectors" deviceset="USB_SOLDER_PADS" device=""/>
 <part name="FRAME2" library="SparkFun-Aesthetics" deviceset="FRAME-LEDGER" device="">
@@
 <wire x1="619.76" y1="99.06" x2="619.76" y2="0" width="0.1524" layer="97" style="longdash"/>
 <wire x1="619.76" y1="99.06" x2="779.78" y2="99.06" width="0.1524" layer="97" style="longdash"/>
-<text x="621.538" y="238.506" size="1.27" layer="97" font="vector" align="center">Digital Decoupling
-Pins 3</text>
 <wire x1="619.76" y1="99.06" x2="619.76" y2="162.56" width="0.2032" layer="97" style="longdash"/>
 <text x="414.02" y="45.72" size="2.54" layer="94" font="vector" align="center">JTAG Connection Points</text>
@@
 </instance>
 <instance part="LOGO1" gate="G$1" x="721.36" y="35.56" smashed="yes"/>
-<instance part="C8" gate="G$1" x="627.38" y="215.9" smashed="yes">
-<attribute name="NAME" x="628.904" y="218.821" size="1.778" layer="95" font="vector"/>
-<attribute name="VALUE" x="628.904" y="213.741" size="1.778" layer="96" font="vector"/>
-</instance>
-<instance part="C9" gate="G$1" x="622.3" y="215.9" smashed="yes">
-<attribute name="NAME" x="618.744" y="218.821" size="1.778" layer="95" font="vector"/>
-<attribute name="VALUE" x="616.204" y="213.741" size="1.778" layer="96" font="vector"/>
-</instance>
-<instance part="GND9" gate="1" x="622.3" y="205.74" smashed="yes">
-<attribute name="VALUE" x="622.3" y="205.486" size="1.778" layer="96" font="vector" align="top-center"/>
-</instance>
-<instance part="SUPPLY3" gate="G$1" x="622.3" y="226.06" smashed="yes">
-<attribute name="VALUE" x="622.3" y="228.854" size="1.778" layer="96" font="vector" align="bottom-center"/>
-</instance>
 <instance part="JP14" gate="JP1" x="398.78" y="243.84" smashed="yes" rot="MR180">
 <attribute name="VALUE" x="386.08" y="251.714" size="1.778" layer="96" font="vector" rot="MR180"/>
@@
 </segment>
 <segment>
-<pinref part="C8" gate="G$1" pin="1"/>
-<wire x1="627.38" y1="220.98" x2="627.38" y2="223.52" width="0.1524" layer="91"/>
-<pinref part="C9" gate="G$1" pin="1"/>
-<wire x1="622.3" y1="220.98" x2="622.3" y2="223.52" width="0.1524" layer="91"/>
-<wire x1="627.38" y1="223.52" x2="622.3" y2="223.52" width="0.1524" layer="91"/>
-<wire x1="622.3" y1="226.06" x2="622.3" y2="223.52" width="0.1524" layer="91"/>
-<junction x="622.3" y="223.52"/>
-<pinref part="SUPPLY3" gate="G$1" pin="3.3V"/>
-</segment>
-<segment>
 <pinref part="SUPPLY14" gate="G$1" pin="3.3V"/>
 <pinref part="R7" gate="G$1" pin="2"/>
@@
 <pinref part="R1" gate="G$1" pin="1"/>
 <wire x1="530.86" y1="30.48" x2="530.86" y2="33.02" width="0.1524" layer="91"/>
-</segment>
-<segment>
-<pinref part="C9" gate="G$1" pin="2"/>
-<pinref part="GND9" gate="1" pin="GND"/>
-<wire x1="622.3" y1="213.36" x2="622.3" y2="210.82" width="0.1524" layer="91"/>
-<pinref part="C8" gate="G$1" pin="2"/>
-<wire x1="622.3" y1="210.82" x2="622.3" y2="208.28" width="0.1524" layer="91"/>
-<wire x1="627.38" y1="213.36" x2="627.38" y2="210.82" width="0.1524" layer="91"/>
-<wire x1="627.38" y1="210.82" x2="622.3" y2="210.82" width="0.1524" layer="91"/>
-<junction x="622.3" y="210.82"/>
 </segment>
 <segment>
@@
 </segment>
 <segment>
-<wire x1="396.24" y1="132.08" x2="391.16" y2="132.08" width="0.1524" layer="91"/>
-<label x="396.24" y="132.08" size="1.27" layer="95" font="vector" xref="yes"/>
-<pinref part="U$2" gate="G$1" pin="5"/>
-</segment>
-<segment>
 <pinref part="R4" gate="G$1" pin="2"/>
 <wire x1="685.8" y1="127" x2="683.26" y2="127" width="0.1524" layer="91"/>
 <label x="683.26" y="127" size="1.27" layer="95" font="vector" rot="MR0" xref="yes"/>
 </segment>
+<segment>
+<wire x1="396.24" y1="129.54" x2="391.16" y2="129.54" width="0.1524" layer="91"/>
+<label x="396.24" y="129.54" size="1.27" layer="95" font="vector" xref="yes"/>
+<pinref part="U$2" gate="G$1" pin="4"/>
+</segment>
 </net>
 <net name="IO6/SDA/I2S_SDO" class="0">
@@
 </segment>
 <segment>
-<wire x1="396.24" y1="129.54" x2="391.16" y2="129.54" width="0.1524" layer="91"/>
-<label x="396.24" y="129.54" size="1.27" layer="95" font="vector" rot="MR180" xref="yes"/>
-<pinref part="U$2" gate="G$1" pin="4"/>
-</segment>
-<segment>
 <pinref part="R3" gate="G$1" pin="1"/>
 <wire x1="721.36" y1="127" x2="723.9" y2="127" width="0.1524" layer="91"/>
 <label x="723.9" y="127" size="1.27" layer="95" font="vector" rot="MR180" xref="yes"/>
 </segment>
-</net>
+<segment>
+<wire x1="396.24" y1="132.08" x2="391.16" y2="132.08" width="0.1524" layer="91"/>
+<label x="396.24" y="132.08" size="1.27" layer="95" font="vector" rot="MR180" xref="yes"/>
+<pinref part="U$2" gate="G$1" pin="5"/>
+</segment>
+</net>
